File: B3_POE/PCB/reCamera_B101_B3_POE.kicad_pcb (KiCad board)
At the start: 4 copper layers, 30 x 30.1 mm, 48 parts, among them J1 ST-BTB-058060-A, K1 TD-1100AP-A4N-D1R, K2 TD-1100AP-A4N-D1R, T1 KHX1631SR, U1 UM10B, U2 XS2100S, U3 SY8502FCC

Commit message: PoE Modified
Parts:
- C3, C4: moved to B.Cu
- R10: value 22k -> 38k
- moved D1 3.53 mm to (100.3, 104.6), turned to 0 degrees
- moved C4 3.44 mm to (113.7, 107.3), turned to 180 degrees
- moved C3 3.33 mm to (107.4, 107.5), turned to 180 degrees
- moved D11 1.43 mm to (107.0, 111.0)
- moved D12 1.11 mm to (113.3, 111.2)
Routing:
- net GND: track 106.8 -> 115.3 mm, vias 59 -> 44
- net /PHYRXP: track 32.2 -> 40.3 mm
- net /PHYTXP: track 23.6 -> 29.8 mm
- net POE_A1: track 29.3 -> 24.1 mm, vias 2 -> 0
- net /PHYRXN: track 35.5 -> 39.0 mm
- net /PHYTXN: track 30.8 -> 33.7 mm
- net EPHY_RXN: track 25.4 -> 27.0 mm
- net Net-(C4-Pad2): track 1.49 -> 2.97 mm, vias 0 -> 1
- net EPHY_TXN: track 43.3 -> 44.5 mm
- net Net-(C3-Pad2): track 1.51 -> 2.25 mm, vias 0 -> 1
- net EPHY_RXP: track 27.4 -> 26.9 mm
