File: B3_POE/PCB/reCamera_B101_B3_POE.kicad_sch (KiCad schematic)
At the start: 48 parts, among them J1 ST-BTB-058060-A, K1 TD-1100AP-A4N-D1R, K2 TD-1100AP-A4N-D1R, T1 KHX1631SR, U1 UM10B, U2 XS2100S, U3 SY8502FCC

Commit message: PoE Modified
Parts:
- R10: value 22k -> 38k
Changed lines of the file:
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@@
 			)
 		)
-		(property "Value" "22k"
+		(property "Value" "38k"
 			(at 333.248 177.038 0)
 			(effects
