File: reCamera_Base_Board/B3_POE/PCB/reCamera 2002 POE Board.kicad_pcb (KiCad board)
At the start: 4 copper layers, 30 x 30 mm, 74 parts, among them J1 ST-BTB-058060-A, J3 1.25-5A-WT, K1 TD-1100AP-A4N-D1R, K2 TD-1100AP-A4N-D1R, T1 KHX1631SR, U3 TPS2121RUXR

Commit message: 更新了三张PCB
Parts:
- removed C1, C14: 22uF, Capacitor:C0805
- removed C15, C22, C23: 100nF, Capacitor:C0402
- removed C8: 1uF, Capacitor:C0402
- removed D10: 27-21/GHC-YR1S2M/3C, Diode:LED2-0.6X1.7MM
- removed R1: 510R, Resistor:R0402
- removed R11: 56K, Resistor:R0402
- removed R15: 8.2K, Resistor:R0402
- removed R22, R26: 19.6K, Resistor:R0402
- removed R23, R25: 20K, Resistor:R0402
- removed R24, R28: 4.7K, Resistor:R0402
- removed R29, R31: 10K, Resistor:R0402
- removed R3: 0R, Resistor:R0805
- removed TP13: Test Point, Misc:TP-D35MIL
- removed U3: TPS2121RUXR, Ic:VQFN12-2.5x2x1mm
- added C49: 10nF, Capacitor:C0402, F.Cu at (109.0, 114.4)
- added C50: 10nF, Capacitor:C0402, F.Cu at (105.6, 103.2)
- added D13: CESD3V3D5, Diode:SOD-523, B.Cu at (123.2, 109.4)
- added D5: CESD3V3D5, Diode:SOD-523, B.Cu at (123.2, 110.6)
- added D6: CESD3V3D5, Diode:SOD-523, B.Cu at (123.2, 111.9)
- added D7: CESD3V3D5, Diode:SOD-523, B.Cu at (123.2, 113.0)
- added D8: CESD3V3D5, Diode:SOD-523, B.Cu at (123.2, 114.2)
- added J5: 1.25-6A-LT, Connector:FPC6-1.25-12.5X3.7X4.65MM, B.Cu at (125.6, 111.3)
- added L1: CMC4532H-102-2P-T, Inductor:INT4-2.2-4.5X3.2X2.8MM, F.Cu at (103.4, 123.7)
- added L3: 300mA, Inductor:INT4-1.45-3.3X2.5X2.5MM, F.Cu at (103.4, 123.7)
- added Q1: CJ3407, Mosfet:SOT23, F.Cu at (110.5, 106.2)
- added Q2: CJ3407, Mosfet:SOT23, F.Cu at (109.6, 111.3)
- added R34: 100K, Resistor:R0402, F.Cu at (108.2, 115.7)
- added R39: 100K, Resistor:R0402, F.Cu at (105.6, 102.5)
- added R40: 100K, Resistor:R0402, F.Cu at (105.6, 100.8)
- added R41: 100R, Resistor:R0402, F.Cu at (107.4, 114.5)
- added R43: 100R, Resistor:R0402, F.Cu at (105.6, 101.7)
- added TP12: Test Point, Misc:TP-D35MIL, B.Cu at (123.0, 117.6)
- added TP15: Test Point, Misc:TP-D35MIL, F.Cu at (111.9, 109.5)
- added TP9: Test Point, Misc:TP-D35MIL, B.Cu at (124.9, 117.6)
- added U10: BC856S, Transistor:SOT-363, F.Cu at (107.6, 102.0)
- added U9: BC856S, Transistor:SOT-363, F.Cu at (105.8, 114.8)
- C12: value 100uF -> 47uF
- J2: value ~ -> ST-FH-254-0106-1*2P-PC3.0
- J4: value ~ -> ST-FH-254-0106-1*4P-PC3.0
- R2: value 0R -> 100K; footprint Resistor:R0805 -> Resistor:R0402
- moved R2 9.71 mm to (108.2, 114.5), turned to 90 degrees
- moved TP11 6.36 mm to (109.5, 108.8)
- moved TP10 2.85 mm to (107.2, 110.8)
- moved R4 0.77 mm to (124.2, 116.0)
- moved R5 0.77 mm to (124.9, 116.0)
- moved TP1 0.51 mm to (128.6, 119.7)
- moved TP2 0.41 mm to (128.6, 122.1)
- moved C12 0.07 mm to (102.7, 108.4)
Connections:
- net /DN renamed /POE Board/DN
- net /DP renamed /POE Board/DP
- net /PHYRXN renamed /POE Board/PHYRXN
- net /PHYRXP renamed /POE Board/PHYRXP
- net /PHYTXN renamed /POE Board/PHYTXN
- net /PHYTXP renamed /POE Board/PHYTXP
- net /POE_VIN-_ModeA renamed /POE Board/POE_VIN-_ModeA
- D4 pad 2: /POE_VIN+_ModeA -> /POE Board/POE_VIN+_ModeA
- R14 pad 2: /POE_VIN+_ModeA -> /POE Board/POE_VIN+_ModeA
- R2 pad 1: /POE_VIN+_ModeA -> GND
- R2 pad 2: Net-(C19-Pad1) -> Net-(Q2-G)
- T1 pad 15: /POE_VIN+_ModeA -> /POE Board/POE_VIN+_ModeA
Routing:
- net /POE Board/POE_VIN+_ModeA: track 0.00 -> 32.6 mm, vias 0 -> 3
- net /POE_VIN+_ModeA: track 30.5 -> 0.00 mm, vias 3 -> 0
- net SDIO_CLK/3V3: track 0.00 -> 15.7 mm, vias 0 -> 1
- net VIN: track 35.9 -> 51.6 mm, vias 12 -> 8
- net SDIO_CMD/3V3: track 0.00 -> 15.1 mm, vias 0 -> 1
- net SDIO_D0/3V3: track 0.00 -> 11.7 mm, vias 0 -> 1
- net Net-(U3-OV1): track 11.3 -> 0.00 mm, vias 2 -> 0
- net Net-(U3-ILM): track 11.0 -> 0.00 mm, vias 2 -> 0
- net Net-(U3-PR1): track 9.92 -> 0.00 mm, vias 2 -> 0
- net SDIO_D1/3V3: track 0.00 -> 9.35 mm, vias 0 -> 1
- net Net-(Q1-G): track 0.00 -> 8.18 mm
- net POE_VOUT_5V: track 1.42 -> 9.00 mm
- net Net-(U3-ST): track 7.30 -> 0.00 mm, vias 2 -> 0
- net SDIO_D3/3V3: track 0.00 -> 7.00 mm, vias 0 -> 1
- net /POE Board/POE_VIN-_ModeA: track 19.7 -> 25.1 mm
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- removed copper zone on F.Cu, net POE_VOUT_5V
- removed copper zone on B.Cu, net VIN
- removed copper zone on F.Cu, net VIN_5V
Other:
- board text added: "GND"
- board text added: "RX"
- board text added: "TX"
- board text added: "v1.2 09/04/25"
- board text removed: "v1.0 07/03/25"
