File: reCamera_Base_Board/B3_POE/PCB/reCamera 2002 POE Board.kicad_sch (KiCad schematic)
At the start: 74 parts, among them J1 ST-BTB-058060-A, J3 1.25-5A-WT, K1 TD-1100AP-A4N-D1R, K2 TD-1100AP-A4N-D1R, T1 KHX1631SR, U3 TPS2121RUXR

Commit message: 更新了三张PCB
Parts:
- removed C1, C14: 22uF, Capacitor:C0805, symbol Seeed_libdb:Capacitors/302013260
- removed C10, C17, C5: 1nF, Capacitor:C1206, symbol libdb:Capacitors/302011962
- removed C11: 100pF, Capacitor:C0402, symbol libdb:Capacitors/302010012
- removed C12, C2: 100uF, Capacitor:C1206, symbol Seeed_libdb:Capacitors/302013339
- removed C13, C15, C22, C23, C3, C4, C7: 100nF, Capacitor:C0402, symbol libdb:Capacitors/302010004
- removed C16, C6: 10uF, Capacitor:C0603, symbol libdb:Capacitors/302010103
- removed C18, C9: 10pF, Capacitor:C0402, symbol libdb:Capacitors/302010001
- removed C19: 10nF, Capacitor:C0603, symbol Seeed_libdb:Capacitors/302012962
- removed C8: 1uF, Capacitor:C0402, symbol Seeed_libdb:Capacitors/302010040
- removed D1: SMF5.0CA, Diode:SOD-123, symbol Seeed_libdb:Diode/304051318
- removed D10: 27-21/GHC-YR1S2M/3C, Diode:LED2-0.6X1.7MM, symbol libdb:Diode/304090030
- removed D11, D12: UDD32C03L01, Diode:SOD-323, symbol libdb:Diode/304060354
- removed D2, D3: ESDPSA0402V05, Diode:ESD-0402, symbol libdb:Diode/304060074
- removed D4: 58V 600W, Diode:DO-214AA-SMB-NONPOLAR, symbol Seeed_libdb:Diode/304050978
- removed F1: 2A, Fuse:F1210, symbol libdb:Fuse/307010043
- removed FB1: 120R, Inductor:L0603, symbol Seeed_libdb:Ferrite Bead/303030024
- removed J1: ST-BTB-058060-A, Connector:BTB60-Male-Female-0.5-17.7x4.4mm, symbol libdb:Connector/320210641
- removed J2: ~, Connector:JST2P-2.54-5.58X2.5X3.5MM, symbol Seeed_libdb:Connector/ST-FH-254-0106-1*2P-PC3.0
- removed J3: 1.25-5A-WT, Connector:JST5_2P_1d25_7_9x4_3x3_4mm, symbol Seeed_libdb:Connector/320112110
- removed J4: ~, Connector:JST4P-2.54-10.66X2.5X3.5MM, symbol Seeed_libdb:Connector/ST-FH-254-0106-1*4P-PC3.0
- removed K1, K2: TD-1100AP-A4N-D1R, Switch:SW5-SMD-4.56X2.3X1.9MM, symbol libdb:Switch/311990111
- removed R1: 510R, Resistor:R0402, symbol libdb:Resistors/301010050
- removed R11: 56K, Resistor:R0402, symbol Seeed_libdb:Resistors/301010032
- removed R12, R7: 5.1K, Resistor:R0402, symbol libdb:Resistors/301010017
- removed R13, R14: 75R, Resistor:R0603, symbol libdb:Resistors/301010269
- removed R15: 8.2K, Resistor:R0402, symbol Seeed_libdb:Resistors/301010024
- removed R16, R17, R8, R9: 0R, Resistor:R0402, symbol Seeed_libdb:Resistors/301010000
- removed R18: 1K, Resistor:R0603, symbol Seeed_libdb:Resistors/301010291
- removed R2, R3: 0R, Resistor:R0805, symbol Seeed_libdb:Resistors/301010359
- removed R22, R26: 19.6K, Resistor:R0402, symbol Seeed_libdb:Resistors/301013446
- removed R23, R25: 20K, Resistor:R0402, symbol Seeed_libdb:Resistors/301010072
- removed R24, R28: 4.7K, Resistor:R0402, symbol Seeed_libdb:Resistors/301010633
- removed R29, R31, R4: 10K, Resistor:R0402, symbol libdb:Resistors/301010047
- removed R5: 20K, Resistor:R0402, symbol libdb:Resistors/301010072
- removed R6: 1M, Resistor:R1206, symbol libdb:Resistors/301010410
- removed T1: KHX1631SR, Misc:TRF_16p_1d27_12d7x7d15x5d1mm, symbol libdb:Misc/303060474
- removed TP1, TP2, TP3: Test Point, Misc:TP-80X40MIL, symbol Seeed_libdb:Misc/TP-80X40MIL
- removed TP10, TP11, TP13, TP4, TP5, TP6, TP8: Test Point, Misc:TP-D35MIL, symbol libdb:Misc/TP35C_SMD
- removed U3: TPS2121RUXR, Ic:VQFN12-2.5x2x1mm, symbol Seeed_libdb:Ic/310032001
- removed USB1: ST-USB-Y3120, Connector:USB2.0-TYPE-C-SMD-12X7.35X3.3MM, symbol libdb:Connector/ST-USB-Y3120
Connections:
- no-connect marks 16 -> 0
Other:
- added sheet 01 Descriptions (01 Descriptions.kicad_sch)
- added sheet POE Board (POE Board.kicad_sch)
- note removed: "Imax=1.2A"
- note removed: "Imax=200mA"
- note removed: "Imax=2A"
- note removed: "Output Current Limit(ILM): ILM = 2.0375A"
- note removed: "Overvoltage Supervisor(OVx): Vin_max = (R22+R24)*Vov/R24 = (19.6K+4.7K)*1.06V/4.7K = 5.5V"
- note removed: "POE Module"
- note removed: "POE_VIN"
- note removed: "POE_VOUT"
- note removed: "Priority Supervisor(PR1): Vin1_min = (R23+R31)*Vov/R31 = (20K+10K)*1.06V/10K = 3.18V"
- note removed: "USB_DET:(1.8V Domain) LOW: USB Host High: USB Device"
